File: Module 3/KiCad/Module 3.kicad_sch (KiCad schematic)
At the start: 19 parts, among them SW1 BLUE_LED, SW2 YELLOW_LED, SW3 GREEN_LED, SW4 RED_LED

Commit message: Added Big Red Button to Module 3
- Created new custom symbol for Big Red Button
- Added the Big Red Button to Module 3 Schematic
- Updated image for Module 3 Schematic
- Updated README file
Parts:
- added SW5: SW_Lock_NC_NO, symbol IEEE_CS_Escape_Room_Symbols_v1:SW_Lock_NC_NO
Connections:
- net GND: now also SW5.3
- net at A1.9 (A0): now also SW5.4
- no-connect marks 1 -> 0
Changed lines of the file:
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@@
+	)
+	(junction
+		(at 90.17 82.55)
+		(diameter 0)
+		(color 0 0 0 1)
 	)
 	(junction
@@
 		(color 0 0 0 1)
 	)
-	(no_connect
-		(at 121.92 110.49)
-	)
 	(wire
 		(pts
@@
 	(wire
 		(pts
+			(xy 114.3 110.49) (xy 121.92 110.49)
+		)
+		(stroke
+			(width 0)
+			(type default)
+			(color 0 132 132 1)
+		)
+	)
+	(wire
+		(pts
 			(xy 147.32 105.41) (xy 158.75 105.41)
 		)
@@
 	(wire
 		(pts
+			(xy 90.17 82.55) (xy 90.17 91.44)
+		)
+		(stroke
+			(width 0)
+			(type default)
+			(color 0 0 0 1)
+		)
+	)
+	(wire
+		(pts
 			(xy 147.32 110.49) (xy 158.75 110.49)
 		)
@@
 	(wire
 		(pts
+			(xy 114.3 82.55) (xy 114.3 110.49)
+		)
+		(stroke
+			(width 0)
+			(type default)
+			(color 0 132 132 1)
+		)
+	)
+	(wire
+		(pts
 			(xy 90.17 110.49) (xy 90.17 116.84)
 		)
@@
 	(wire
 		(pts
+			(xy 106.68 82.55) (xy 114.3 82.55)
+		)
+		(stroke
+			(width 0)
+			(type default)
+			(color 0 132 132 1)
+		)
+	)
+	(wire
+		(pts
 			(xy 194.31 73.66) (xy 200.66 73.66)
 		)
@@
 	(wire
 		(pts
-			(xy 90.17 88.9) (xy 90.17 91.44)
+			(xy 90.17 80.01) (xy 90.17 82.55)
 		)
 		(stroke
@@
 			(width 0)
 			(type default)
+		)
+	)
+	(wire
+		(pts
+			(xy 90.17 82.55) (xy 96.52 82.55)
+		)
+		(stroke
+			(width 0)
+			(type default)
+			(color 0 0 0 1)
 		)
 	)
@@
 	)
 	(symbol
+		(lib_id "IEEE_CS_Escape_Room_Symbols_v1:SW_Lock_NC_NO")
+		(at 101.6 78.74 0)
+		(unit 1)
+		(body_style 1)
+		(exclude_from_sim no)
+		(in_bom yes)
+		(on_board yes)
+		(in_pos_files yes)
+		(dnp no)
+		(fields_autoplaced yes)
+		(property "Reference" "SW5"
+			(at 101.6 69.85 0)
+			(show_name no)
+			(do_not_autoplace no)
+			(effects
+				(font
+					(size 1.27 1.27)
+				)
+			)
+		)
+		(property "Value" "SW_Lock_NC_NO"
+			(at 101.6 72.39 0)
+			(show_name no)
+			(do_not_autoplace no)
+			(effects
+				(font
+					(size 1.27 1.27)
+				)
+			)
+		)
+		(property "Footprint" ""
+			(at 101.6 78.74 0)
+			(hide yes)
+			(show_name no)
+			(do_not_autoplace no)
+			(effects
+				(font
+					(size 1.27 1.27)
+				)
+			)
+		)
+		(property "Datasheet" "https://www.amazon.com/dp/B0068AGC2Q"
+			(at 101.6 85.852 0)
+			(hide yes)
+			(show_name no)
+			(do_not_autoplace no)
+			(effects
+				(font
+					(size 1.27 1.27)
+				)
+			)
+		)
+		(property "Description" "Big red emergency button that locks when pressed and needs a key to be released. It has 2 rails, one is normally closed and the other is normally open."
+			(at 101.6 88.138 0)
+			(hide yes)
+			(show_name no)
+			(do_not_autoplace no)
+			(effects
+				(font
+					(size 1.27 1.27)
+				)
+			)
+		)
+		(pin "3"
+		)
+		(pin "2"
+		)
+		(pin "4"
+		)
+		(pin "1"
+		)
+		(instances
+			(project "Module 3"
+				(path "/6b1920bf-1ae7-482d-afb4-9147762c4aed"
+					(reference "SW5")
+					(unit 1)
+				)
+			)
+		)
+	)
+	(symbol
 		(lib_id "power:GND")
 		(at 200.66 102.87 270)
@@
 	(symbol
 		(lib_id "power:GND")
-		(at 90.17 88.9 180)
+		(at 90.17 80.01 180)
 		(unit 1)
 		(body_style 1)
@@
 		(dnp no)
 		(property "Reference" "#PWR01"
-			(at 90.17 82.55 0)
+			(at 90.17 73.66 0)
 			(hide yes)
 			(show_name no)
@@
 		)
 		(property "Value" "GND"
-			(at 90.17 84.836 0)
+			(at 90.17 75.946 0)
 			(show_name no)
 			(do_not_autoplace no)
@@
 		)
 		(property "Footprint" ""
-			(at 90.17 88.9 0)
+			(at 90.17 80.01 0)
 			(hide yes)
 			(show_name no)
@@
 		)
 		(property "Datasheet" ""
-			(at 90.17 88.9 0)
+			(at 90.17 80.01 0)
 			(hide yes)
 			(show_name no)
@@
 		)
 		(property "Description" "Power symbol creates a global label with name \"GND\" , ground"
-			(at 90.17 88.9 0)
-			(hide yes)
-			(show_name no)
+			(at 90.17 80.01 0)
+			(hide yes)
+			(show_name no)
