File: KiCad/Module 3/Module 3.kicad_sch (KiCad schematic)
At the start: 21 parts, among them SW1 BLUE_LED, SW2 YELLOW_LED, SW3 GREEN_LED, SW4 RED_LED, SW5 SW_Lock_NC_NO, SW6 RED_LED

Commit message: Swapped names of SW5 and SW6 in Module 3 schematic
Swapped names of SW5 and SW6 in Module 3 schematic so all five button LEDs are named SW1-SW5 instead of SW1-SW4 and SW6.
Parts:
- renumbered SW6 to SW5, SW5 to SW6
Changed lines of the file:
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@@
 		(dnp no)
 		(fields_autoplaced yes)
-		(property "Reference" "SW5"
+		(property "Reference" "SW6"
 			(at 92.71 67.31 0)
 			(show_name no)
@@
 			(project "Module 3"
 				(path "/6b1920bf-1ae7-482d-afb4-9147762c4aed"
-					(reference "SW5")
+					(reference "SW6")
 					(unit 1)
 				)
@@
 		(in_pos_files yes)
 		(dnp no)
-		(property "Reference" "SW6"
+		(property "Reference" "SW5"
 			(at 165.1 108.204 0)
 			(show_name no)
@@
 			(project "Module 3"
 				(path "/6b1920bf-1ae7-482d-afb4-9147762c4aed"
-					(reference "SW6")
-					(unit 1)
-				)
+					(reference "SW5")
+					(unit 1)
+				)
